Commit message: Hi

File: src/marc/urdf/marc.urdf (robot description, URDF)
Before this commit: robot marc, 9 links, 8 joints
Links:
- removed link ee_rotation_x_link
- removed link ee_rotation_y_link
- removed link ee_rotation_z_link
- added link ee_rotation_x
- added link ee_rotation_y
- added link robot_ee
Joints:
- joint ee_rotation_joint_x: child ee_rotation_x_link -> ee_rotation_x; limit lower=-3.14 upper=3.14 effort=5 velocity=1 -> lower=-3.1416 upper=3.1416 effort=1 velocity=1
- joint ee_rotation_joint_y: child ee_rotation_y_link -> ee_rotation_y; limit lower=-3.14 upper=3.14 effort=5 velocity=1 -> lower=-3.1416 upper=3.1416 effort=1 velocity=1; parent ee_rotation_x_link -> ee_rotation_x
- joint ee_rotation_joint_z: child ee_rotation_z_link -> robot_ee; limit lower=-3.14 upper=3.14 effort=5 velocity=1 -> lower=-3.1416 upper=3.1416 effort=1 velocity=1; parent ee_rotation_y_link -> ee_rotation_y
