Commit message: Changes

File: install/arm_config/share/arm_config/config/marc.ros2_control.xacro (robot description, xacro)
@@ -38,8 +38,8 @@
                 </state_interface>
             </joint>
-            <joint name="ee_rotation_joint_y">
+            <joint name="ee_rotation_joint_z">
                 <command_interface name="position"/>
                 <state_interface name="position">
-                  <param name="initial_value">${initial_positions['ee_rotation_joint_y']}</param>
+                  <param name="initial_value">${initial_positions['ee_rotation_joint_z']}</param>
                 </state_interface>
             </joint>

File: install/marc/share/marc/urdf/marc.urdf (robot description, URDF)
Before this commit: robot marc, 9 links, 8 joints
Links:
- removed link ee_rotation_y
- added link ee_rotation_z
Joints:
- removed joint ee_rotation_joint_y
- added joint ee_rotation_joint_z: type revolute, parent ee_rotation_x, child ee_rotation_z, origin xyz=0 0 0 rpy=0 0 0, axis 0 0 1, limit lower=-3.1416 upper=3.1416 effort=10.5 velocity=1.5
- joint ee_rotation_joint_x: limit lower=-3.1416 upper=3.1416 effort=1 velocity=1 -> lower=-3.1416 upper=3.1416 effort=10.5 velocity=1.5
